File: Dimmer3.kicad_pcb (KiCad board)
At the start: 2 copper layers, 57.7 x 56 mm, 63 parts, among them IC1 TMAG3001A1YBGR, J1 Conn_02x06_Odd_Even, SW1 SW_Push, SW2 SW_Push, SW3 SW_Push, SW4 SW_Push, SW5 SW_Push, U1 STM32WB5MMGH6TR

Commit message: modified debug port
Parts:
- C10, C12, C21, C22, C3, C4, C5, C6, C7, C8, C9: value 100n/1608 -> 100nF/1608
- C11: value 4.7u/1608 -> 4.7uF/1608
- C13, C14, C15, C16, C17, C18, C19, C20: value 1u/1608 -> 1uF/1608
Connections:
- J1 pad 10: /LPUART_TXD -> /NRST
- J1 pad 12: /NRST -> /LPUART_TXD
- J1 pad 2: /SWCLK -> /SWDIO
- J1 pad 4: /SWDIO -> /SWCLK
- U1 pad 12: /LPUART_TXD -> /LPUART_RXD
- U1 pad 9: /LPUART_RXD -> /LPUART_TXD
Routing:
- net /LPUART_RXD: track 14.8 -> 13.2 mm
- net /LPUART_TXD: track 10.9 -> 12.4 mm
- net /SWDIO: track 16.6 -> 18.0 mm
- net GND: track 54.0 -> 55.2 mm, vias 270 -> 273
- net /NRST: track 18.1 -> 19.1 mm
- net /SWCLK: track 19.2 -> 18.3 mm, vias 1 -> 0
