File: Dimmer3.kicad_sch (KiCad schematic)
At the start: 63 parts, among them IC1 TMAG3001A1YBGR, J1 Conn_02x06_Odd_Even, SW1 SW_Push, SW2 SW_Push, SW3 SW_Push, SW4 SW_Push, SW5 SW_Push, U1 STM32WB5MMGH6TR

Commit message: modified debug port
Connections:
- net LPUART_RXD: now also U1.12 (PC0); no longer U1.9 (PC1)
- net LPUART_TXD: now also J1.12 (Pin_12), U1.9 (PC1); no longer J1.10 (Pin_10), U1.12 (PC0)
- net NRST: now also J1.10 (Pin_10); no longer J1.12 (Pin_12)
- net SWCLK: now also J1.4 (Pin_4); no longer J1.2 (Pin_2)
- net SWDIO: now also J1.2 (Pin_2); no longer J1.4 (Pin_4)
Changed lines of the file:
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@@
 	)
 	(label "SWDIO"
-		(at 196.85 264.16 180)
+		(at 196.85 261.62 180)
 		(effects
 			(font
@@
 	)
 	(label "LPUART_TXD"
-		(at 196.85 271.78 180)
+		(at 196.85 274.32 180)
 		(effects
 			(font
@@
 	)
 	(label "SWCLK"
-		(at 196.85 261.62 180)
+		(at 196.85 264.16 180)
 		(effects
 			(font
@@
 	)
 	(label "NRST"
-		(at 196.85 274.32 180)
+		(at 196.85 271.78 180)
 		(effects
 			(font
@@
 	)
 	(label "LPUART_TXD"
-		(at 40.64 193.04 0)
+		(at 40.64 195.58 0)
 		(effects
 			(font
@@
 	)
 	(label "LPUART_RXD"
-		(at 40.64 195.58 0)
-		(effects
-			(font
+		(at 40.64 193.04 0)
+		(effects
+			(font
